File: Shield/Canbus-proto2.brd (EAGLE design)
At the start: 92.1 x 52.7 mm, 81 parts, among them J1 Digital_0_7, J2 Analog, J3 Digital_8_13, J4 Analog, J5 Digital_14_21

Commit message: Updated canbus board to fix a layout issue, updated DueD to use DC/DC converter
Connections:
- net D14_TX3: now also J5.1, SL5.1; no longer J5.8, SL5.8
- net D15_RX3: now also J5.2, SL5.2; no longer J5.7, SL5.7
- net D16_TX2: now also J5.3, SL5.3; no longer J5.6, SL5.6
- net D17_RX2: now also J5.4, SL5.4; no longer J5.5, SL5.5
- net D18_TX1: now also J5.5, SL5.5; no longer J5.4, SL5.4
- net D19_RX1: now also J5.6, SL5.6; no longer J5.3, SL5.3
- net D20_SDA: now also J5.7, SL5.7; no longer J5.2, SL5.2
- net D21_SCL: now also J5.8, SL5.8; no longer J5.1, SL5.1
Routing:
- net D21_SCL: track 26.0 -> 9.60 mm
- net D20_SDA: track 20.4 -> 11.7 mm
- net D18_TX1: track 19.4 -> 18.3 mm
Changed lines of the file:
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@@
 <wire x1="77.47" y1="2.54" x2="77.47" y2="7.62" width="0.6096" layer="1"/>
 </signal>
-<signal name="D14_TX3">
-<contactref element="SL5" pad="8"/>
-<contactref element="J5" pad="8"/>
-<wire x1="77.47" y1="45.72" x2="77.47" y2="50.8" width="0.6096" layer="1"/>
-</signal>
-<signal name="D15_RX3">
-<contactref element="SL5" pad="7"/>
-<contactref element="J5" pad="7"/>
-<wire x1="74.93" y1="45.72" x2="74.93" y2="50.8" width="0.6096" layer="1"/>
-</signal>
-<signal name="D16_TX2">
+<signal name="D19_RX1">
 <contactref element="SL5" pad="6"/>
 <contactref element="J5" pad="6"/>
@@
 </signal>
 <signal name="D18_TX1">
-<contactref element="SL5" pad="4"/>
-<contactref element="J5" pad="4"/>
-<wire x1="67.31" y1="45.72" x2="67.31" y2="50.8" width="0.6096" layer="1"/>
 <contactref element="U$6" pad="PIN7"/>
-<wire x1="67.31" y1="45.72" x2="69.85" y2="43.18" width="0.254" layer="16"/>
-<wire x1="69.85" y1="43.18" x2="69.85" y2="40.64" width="0.254" layer="16"/>
 <wire x1="69.85" y1="40.64" x2="70.485" y2="40.005" width="0.254" layer="16"/>
 <wire x1="70.485" y1="40.005" x2="71.755" y2="40.005" width="0.254" layer="16"/>
@@
 <via x="72.39" y="36.195" extent="1-16" drill="0.5"/>
 <wire x1="70.485" y1="36.35375" x2="72.39" y2="36.195" width="0.254" layer="1"/>
-</signal>
-<signal name="D17_RX2">
 <contactref element="SL5" pad="5"/>
 <contactref element="J5" pad="5"/>
 <wire x1="69.85" y1="45.72" x2="69.85" y2="50.8" width="0.6096" layer="1"/>
-</signal>
-<signal name="D19_RX1">
+<wire x1="69.85" y1="40.64" x2="69.85" y2="45.72" width="0.254" layer="16"/>
+</signal>
+<signal name="D16_TX2">
 <contactref element="SL5" pad="3"/>
 <contactref element="J5" pad="3"/>
@@
 </signal>
 <signal name="D20_SDA">
-<contactref element="SL5" pad="2"/>
-<contactref element="J5" pad="2"/>
-<wire x1="62.23" y1="45.72" x2="62.23" y2="50.8" width="0.6096" layer="1"/>
 <contactref element="R24" pad="2"/>
 <contactref element="U$6" pad="PIN5"/>
 <wire x1="68.16" y1="39.37" x2="69.85" y2="39.37" width="0.254" layer="1"/>
 <wire x1="69.85" y1="39.37" x2="70.485" y2="38.89375" width="0.254" layer="1"/>
-<wire x1="62.23" y1="45.72" x2="64.77" y2="43.18" width="0.254" layer="16"/>
-<wire x1="64.77" y1="43.18" x2="64.77" y2="38.1" width="0.254" layer="16"/>
 <via x="64.77" y="38.1" extent="1-16" drill="0.5"/>
 <wire x1="64.77" y1="38.1" x2="67.31" y2="38.1" width="0.254" layer="1"/>
@@
 <wire x1="67.945" y1="38.735" x2="67.945" y2="39.155" width="0.254" layer="1"/>
 <wire x1="67.945" y1="39.155" x2="68.16" y2="39.37" width="0.254" layer="1"/>
+<contactref element="SL5" pad="7"/>
+<contactref element="J5" pad="7"/>
+<wire x1="74.93" y1="45.72" x2="74.93" y2="50.8" width="0.6096" layer="1"/>
+<wire x1="69.85" y1="39.37" x2="74.93" y2="45.72" width="0" layer="19" extent="1-1"/>
 </signal>
 <signal name="D21_SCL">
-<contactref element="SL5" pad="1"/>
-<contactref element="J5" pad="1"/>
-<wire x1="59.69" y1="45.72" x2="59.69" y2="50.8" width="0.6096" layer="1"/>
 <contactref element="R23" pad="2"/>
 <contactref element="U$6" pad="PIN6"/>
@@
 <wire x1="68.58" y1="36.83" x2="69.215" y2="37.465" width="0.254" layer="1"/>
 <wire x1="69.215" y1="37.465" x2="70.485" y2="37.62375" width="0.254" layer="1"/>
-<wire x1="59.69" y1="45.72" x2="59.69" y2="39.37" width="0.254" layer="16"/>
-<wire x1="59.69" y1="39.37" x2="64.135" y2="34.925" width="0.254" layer="16"/>
-<wire x1="64.135" y1="34.925" x2="67.945" y2="34.925" width="0.254" layer="16"/>
 <via x="67.945" y="34.925" extent="1-16" drill="0.5"/>
 <wire x1="68.16" y1="36.83" x2="68.16" y2="36.0925" width="0.254" layer="1"/>
 <wire x1="68.16" y1="36.0925" x2="67.945" y2="34.925" width="0.254" layer="1"/>
+<contactref element="SL5" pad="8"/>
+<contactref element="J5" pad="8"/>
+<wire x1="77.47" y1="45.72" x2="77.47" y2="50.8" width="0.6096" layer="1"/>
+<wire x1="70.485" y1="37.62375" x2="77.47" y2="45.72" width="0" layer="19" extent="1-1"/>
 </signal>
 <signal name="D22">
@@
 <wire x1="9.906" y1="45.72" x2="9.906" y2="50.8" width="0.6096" layer="1"/>
 </signal>
+<signal name="D17_RX2">
+<contactref element="SL5" pad="4"/>
+<contactref element="J5" pad="4"/>
+<wire x1="67.31" y1="45.72" x2="67.31" y2="50.8" width="0.6096" layer="1"/>
+</signal>
+<signal name="D15_RX3">
+<contactref element="SL5" pad="2"/>
+<contactref element="J5" pad="2"/>
+<wire x1="62.23" y1="45.72" x2="62.23" y2="50.8" width="0.6096" layer="1"/>
+</signal>
+<signal name="D14_TX3">
+<contactref element="SL5" pad="1"/>
+<contactref element="J5" pad="1"/>
+<wire x1="59.69" y1="45.72" x2="59.69" y2="50.8" width="0.6096" layer="1"/>
+</signal>
 </signals>
