File: Shield/canbus-proto2.sch (EAGLE design)
At the start: 81 parts, among them J1 Digital_0_7, J2 Analog, J3 Digital_8_13, J4 Analog, J5 Digital_14_21

Commit message: Switched all passives to 0603 to harmonize part sizes.
Parts:
- C1, C2: value 100nF 0805 -> 100nF; device SparkFun:CAP0805-LARGE -> SparkFun-Passives:CAP0603-CAP
- LED1: value RED 0805 -> RED; device SparkFun:LED0805-LARGE -> SparkFun-LED:LED-RED0603
- LED2: value GREEN 0805 -> GREEN; device SparkFun:LED0805-LARGE -> SparkFun-LED:LED-GREEN0603
- R1, R2: value 1K 0805 -> 1K; device SparkFun:RESISTOR0805-LARGE -> rcl:R-US_R0603
Changed lines of the file:
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@@
 <part name="SL3" library="SparkFun-Connectors" deviceset="M10" device="&quot;" value="Digital_8_13"/>
 <part name="SL1" library="SparkFun" deviceset="M08" device="" value="Digital_0_7"/>
-<part name="C1" library="SparkFun" deviceset="CAP" device="0805-LARGE" value="100nF 0805"/>
-<part name="C2" library="SparkFun" deviceset="CAP" device="0805-LARGE" value="100nF 0805"/>
-<part name="LED1" library="SparkFun" deviceset="LED" device="0805-LARGE" value="RED 0805"/>
-<part name="LED2" library="SparkFun" deviceset="LED" device="0805-LARGE" value="GREEN 0805"/>
-<part name="R1" library="SparkFun" deviceset="RESISTOR" device="0805-LARGE" value="1K 0805"/>
-<part name="R2" library="SparkFun" deviceset="RESISTOR" device="0805-LARGE" value="1K 0805"/>
+<part name="C1" library="SparkFun-Passives" deviceset="CAP" device="0603-CAP" value="100nF"/>
+<part name="C2" library="SparkFun-Passives" deviceset="CAP" device="0603-CAP" value="100nF"/>
+<part name="LED1" library="SparkFun-LED" deviceset="LED-RED" device="0603" value="RED"/>
+<part name="LED2" library="SparkFun-LED" deviceset="LED-GREEN" device="0603" value="GREEN"/>
+<part name="R1" library="rcl" deviceset="R-US_" device="R0603" value="1K"/>
+<part name="R2" library="rcl" deviceset="R-US_" device="R0603" value="1K"/>
 <part name="S1" library="SparkFun" deviceset="TAC_SWITCH" device="PTH" value="RESET"/>
 <part name="GND1" library="SparkFun" deviceset="GND" device=""/>
@@
 <instance part="C2" gate="G$1" x="180.34" y="71.12" smashed="yes">
 <attribute name="NAME" x="171.704" y="71.501" size="1.778" layer="95"/>
-<attribute name="VALUE" x="161.544" y="68.961" size="1.778" layer="96"/>
+<attribute name="VALUE" x="171.704" y="68.961" size="1.778" layer="96"/>
 </instance>
 <instance part="LED1" gate="G$1" x="25.4" y="142.24" smashed="yes" rot="R90">

Commit message: Updated canbus board to be more correct, fixed size of ampseal connector, totally new DueD board.
Connections:
- removed net 3V3: POWER.2, SLP.2
- net +3V3: now also POWER.2, SLP.2
Changed lines of the file:
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@@
-</segment>
-</net>
-<net name="3V3" class="0">
-<segment>
-<wire x1="22.86" y1="83.82" x2="35.56" y2="83.82" width="0.1524" layer="91"/>
-<label x="25.4" y="83.82" size="1.778" layer="95"/>
-<pinref part="POWER" gate="G$1" pin="2"/>
-<pinref part="SLP" gate="G$1" pin="2"/>
 </segment>
 </net>
@@
 <pinref part="JP38" gate="G$1" pin="15"/>
 </segment>
-</net>
+<segment>
+<wire x1="22.86" y1="83.82" x2="35.56" y2="83.82" width="0.1524" layer="91"/>
+<label x="25.4" y="83.82" size="1.778" layer="95"/>
+<pinref part="POWER" gate="G$1" pin="2"/>
+<pinref part="SLP" gate="G$1" pin="2"/>
+</segment>
+</net>

Commit message: Updated canbus board to fix a layout issue, updated DueD to use DC/DC converter
Connections:
- net D14_TX3: now also J5.1, SL5.1; no longer J5.8, SL5.8
- net D15_RX3: now also J5.2, SL5.2; no longer J5.7, SL5.7
- net D16_TX2: now also J5.3, SL5.3; no longer J5.6, SL5.6
- net D17_RX2: now also J5.4, SL5.4; no longer J5.5, SL5.5
- net D18_TX1: now also J5.5, SL5.5; no longer J5.4, SL5.4
- net D19_RX1: now also J5.6, SL5.6; no longer J5.3, SL5.3
- net D20_SDA: now also J5.7, SL5.7; no longer J5.2, SL5.2
- net D21_SCL: now also J5.8, SL5.8; no longer J5.1, SL5.1
Changed lines of the file:
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@@
 </segment>
 </net>
-<net name="D14_TX3" class="0">
-<segment>
-<wire x1="208.28" y1="83.82" x2="223.52" y2="83.82" width="0.2032" layer="91"/>
-<label x="210.82" y="83.82" size="1.778" layer="95"/>
-<pinref part="SL5" gate="G$1" pin="8"/>
-<pinref part="J5" gate="G$1" pin="8"/>
-</segment>
-</net>
-<net name="D15_RX3" class="0">
-<segment>
-<wire x1="208.28" y1="81.28" x2="223.52" y2="81.28" width="0.2032" layer="91"/>
-<label x="210.82" y="81.28" size="1.778" layer="95"/>
-<pinref part="SL5" gate="G$1" pin="7"/>
-<pinref part="J5" gate="G$1" pin="7"/>
-</segment>
-</net>
-<net name="D16_TX2" class="0">
+<net name="D19_RX1" class="0">
 <segment>
 <wire x1="208.28" y1="78.74" x2="223.52" y2="78.74" width="0.2032" layer="91"/>
@@
 <net name="D18_TX1" class="0">
 <segment>
-<wire x1="208.28" y1="73.66" x2="223.52" y2="73.66" width="0.2032" layer="91"/>
-<label x="210.82" y="73.66" size="1.778" layer="95"/>
-<pinref part="SL5" gate="G$1" pin="4"/>
-<pinref part="J5" gate="G$1" pin="4"/>
-</segment>
-<segment>
 <pinref part="U$6" gate="G$1" pin="WC"/>
 <wire x1="137.16" y1="-63.5" x2="154.94" y2="-63.5" width="0.1524" layer="91"/>
 </segment>
-</net>
-<net name="D17_RX2" class="0">
 <segment>
 <wire x1="208.28" y1="76.2" x2="223.52" y2="76.2" width="0.2032" layer="91"/>
@@
 </segment>
 </net>
-<net name="D19_RX1" class="0">
+<net name="D16_TX2" class="0">
 <segment>
 <wire x1="208.28" y1="71.12" x2="223.52" y2="71.12" width="0.2032" layer="91"/>
@@
 </net>
 <net name="D20_SDA" class="0">
-<segment>
-<wire x1="208.28" y1="68.58" x2="223.52" y2="68.58" width="0.2032" layer="91"/>
-<label x="210.82" y="68.58" size="1.778" layer="95"/>
-<pinref part="SL5" gate="G$1" pin="2"/>
-<pinref part="J5" gate="G$1" pin="2"/>
-</segment>
 <segment>
 <pinref part="R24" gate="G$1" pin="2"/>
@@
 <wire x1="149.86" y1="-73.66" x2="137.16" y2="-73.66" width="0.1524" layer="91"/>
 </segment>
+<segment>
+<wire x1="208.28" y1="81.28" x2="223.52" y2="81.28" width="0.2032" layer="91"/>
+<label x="210.82" y="81.28" size="1.778" layer="95"/>
+<pinref part="SL5" gate="G$1" pin="7"/>
+<pinref part="J5" gate="G$1" pin="7"/>
+</segment>
 </net>
 <net name="D21_SCL" class="0">
-<segment>
-<wire x1="208.28" y1="66.04" x2="223.52" y2="66.04" width="0.2032" layer="91"/>
-<label x="210.82" y="66.04" size="1.778" layer="95"/>
-<pinref part="SL5" gate="G$1" pin="1"/>
-<pinref part="J5" gate="G$1" pin="1"/>
-</segment>
 <segment>
 <pinref part="R23" gate="G$1" pin="2"/>
@@
 <wire x1="149.86" y1="-66.04" x2="149.86" y2="-68.58" width="0.1524" layer="91"/>
 <wire x1="149.86" y1="-68.58" x2="137.16" y2="-68.58" width="0.1524" layer="91"/>
+</segment>
+<segment>
+<wire x1="208.28" y1="83.82" x2="223.52" y2="83.82" width="0.2032" layer="91"/>
+<label x="210.82" y="83.82" size="1.778" layer="95"/>
+<pinref part="SL5" gate="G$1" pin="8"/>
+<pinref part="J5" gate="G$1" pin="8"/>
 </segment>
 </net>
@@
 </segment>
 </net>
+<net name="D17_RX2" class="0">
+<segment>
+<wire x1="208.28" y1="73.66" x2="223.52" y2="73.66" width="0.2032" layer="91"/>
+<label x="210.82" y="73.66" size="1.778" layer="95"/>
+<pinref part="SL5" gate="G$1" pin="4"/>
+<pinref part="J5" gate="G$1" pin="4"/>
+</segment>
+</net>
+<net name="D15_RX3" class="0">
+<segment>
+<wire x1="208.28" y1="68.58" x2="223.52" y2="68.58" width="0.2032" layer="91"/>
+<label x="210.82" y="68.58" size="1.778" layer="95"/>
+<pinref part="SL5" gate="G$1" pin="2"/>
+<pinref part="J5" gate="G$1" pin="2"/>
+</segment>
+</net>
+<net name="D14_TX3" class="0">
+<segment>
+<wire x1="208.28" y1="66.04" x2="223.52" y2="66.04" width="0.2032" layer="91"/>
+<label x="210.82" y="66.04" size="1.778" layer="95"/>
+<pinref part="SL5" gate="G$1" pin="1"/>
+<pinref part="J5" gate="G$1" pin="1"/>
+</segment>
+</net>
